File: 1_2og_repro.kicad_pcb (KiCad board)
At the start: 2 copper layers, 347.1 x 119.3 mm, 218 parts, among them J1 Conn_01x03, J2 USB_B_Mini, J3 Conn_01x03, Q1 2N7002, SW1 MX_SW_solder, SW10 MX_SW_solder, SW11 MX_SW_solder, SW12 MX_SW_solder, SW13 MX_SW_solder, SW14 MX_SW_solder, SW15 MX_SW_solder, SW16 MX_SW_solder, SW17 MX_SW_solder, SW18 MX_SW_solder, SW19 MX_SW_solder, SW2 MX_SW_solder, SW20 MX_SW_solder, SW21 MX_SW_solder, SW22 MX_SW_solder, SW23 MX_SW_solder, SW24 MX_SW_solder, SW25 MX_SW_solder, SW26 MX_SW_solder, SW27 MX_SW_solder, SW28 MX_SW_solder, SW29 MX_SW_solder, SW3 MX_SW_solder, SW30 MX_SW_solder, SW31 MX_SW_solder, SW32 MX_SW_solder, SW33 MX_SW_solder, SW34 MX_SW_solder, SW35 MX_SW_solder, SW36 MX_SW_solder, SW37 MX_SW_solder, SW38 MX_SW_solder, SW39 MX_SW_solder, SW4 MX_SW_solder, SW40 MX_SW_solder, SW41 MX_SW_solder, SW42 MX_SW_solder, SW43 MX_SW_solder, SW44 MX_SW_solder, SW45 MX_SW_solder, SW46 MX_SW_solder, SW47 MX_SW_solder, SW48 MX_SW_solder, SW49 MX_SW_solder, SW5 MX_SW_solder, SW50 MX_SW_solder, SW51 MX_SW_solder, SW52 MX_SW_solder, SW53 MX_SW_solder, SW54 MX_SW_solder, SW55 MX_SW_solder, SW56 MX_SW_solder, SW57 MX_SW_solder, SW58 MX_SW_solder, SW59 MX_SW_solder, SW6 MX_SW_solder, SW60 MX_SW_solder, SW61 MX_SW_solder, SW62 MX_SW_solder, SW63 MX_SW_solder, SW64 MX_SW_solder, SW65 MX_SW_solder, SW66 MX_SW_solder, SW67 MX_SW_solder, SW68 MX_SW_solder, SW69 MX_SW_solder, SW7 MX_SW_solder, SW70 MX_SW_solder, SW71 MX_SW_solder, SW72 MX_SW_solder, SW73 MX_SW_solder, SW74 MX_SW_solder, SW75 MX_SW_solder, SW76 MX_SW_solder, SW77 MX_SW_solder, SW78 MX_SW_solder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

Commit message: add lightbar kinda (gerbers have not been fully updated yet, bom is broken)
Parts:
- removed REF**: SolderWirePad_1x01_SMD_5x10mm, Connector_Wire:SolderWirePad_1x01_SMD_5x10mm
- J1: footprint Connector_JST:JST_PH_S3B-PH-K_1x03_P2.00mm_Horizontal -> Connector_Molex:Molex_Pico-EZmate_78171-0003_1x03-1MP_P1.20mm_Vertical; moved to B.Cu
- moved J1 2.91 mm to (349.4, 103.5), turned to -90 degrees
Connections:
- J1 pad 1: GND -> +5V
- J1 pad 3: +5V -> GND
Routing:
- net GND: track 65.2 -> 61.7 mm
- net COL6: track 319.7 -> 318.9 mm, vias 2 -> 0
- net COL2: track 397.6 -> 397.0 mm, vias 2 -> 0
- net COL0: track 441.2 -> 441.5 mm, vias 2 -> 0
- net COL1: track 394.8 -> 394.9 mm, vias 2 -> 0
- net +3V3: track 337.3 -> 337.2 mm, vias 10 -> 8
- net ROW4: track 385.6 -> 385.7 mm, vias 2 -> 4

Commit message: dual jst-ph and ezmate support on pcb
Parts:
- added J4: Conn_01x03, Connector_JST:JST_PH_S3B-PH-K_1x03_P2.00mm_Horizontal, F.Cu at (347.7, 105.5)
- moved J1 2.91 mm to (352.3, 103.5)
Routing:
- net GND: track 61.7 -> 76.8 mm, vias 24 -> 28
- net RGB_DB: track 57.2 -> 60.2 mm
- net +5V: track 126.6 -> 129.5 mm
