File: pcb/1_2og_repro.kicad_pcb (KiCad board)
At the start: 2 copper layers, 347.1 x 119.3 mm, 225 parts, among them J1 Pico EzMate, J2 548190519, J3 RAW, J4 S3B, Q1 2N7002, SW1 MX_SW_solder, SW10 MX_SW_solder, SW11 MX_SW_solder, SW12 MX_SW_solder, SW13 MX_SW_solder, SW14 MX_SW_solder, SW15 MX_SW_solder, SW16 MX_SW_solder, SW17 MX_SW_solder, SW18 MX_SW_solder, SW19 MX_SW_solder, SW2 MX_SW_solder, SW20 MX_SW_solder, SW21 MX_SW_solder, SW22 MX_SW_solder, SW23 MX_SW_solder, SW24 MX_SW_solder, SW25 MX_SW_solder, SW26 MX_SW_solder, SW27 MX_SW_solder, SW28 MX_SW_solder, SW29 MX_SW_solder, SW3 MX_SW_solder, SW30 MX_SW_solder, SW31 MX_SW_solder, SW32 MX_SW_solder, SW33 MX_SW_solder, SW34 MX_SW_solder, SW35 MX_SW_solder, SW36 MX_SW_solder, SW37 MX_SW_solder, SW38 MX_SW_solder, SW39 MX_SW_solder, SW4 MX_SW_solder, SW40 MX_SW_solder, SW41 MX_SW_solder, SW42 MX_SW_solder, SW43 MX_SW_solder, SW44 MX_SW_solder, SW45 MX_SW_solder, SW46 MX_SW_solder, SW47 MX_SW_solder, SW48 MX_SW_solder, SW49 MX_SW_solder, SW5 MX_SW_solder, SW50 MX_SW_solder, SW51 MX_SW_solder, SW52 MX_SW_solder, SW53 MX_SW_solder, SW54 MX_SW_solder, SW55 MX_SW_solder, SW56 MX_SW_solder, SW57 MX_SW_solder, SW58 MX_SW_solder, SW59 MX_SW_solder, SW6 MX_SW_solder, SW60 MX_SW_solder, SW61 MX_SW_solder, SW62 MX_SW_solder, SW63 MX_SW_solder, SW64 MX_SW_solder, SW65 MX_SW_solder, SW66 MX_SW_solder, SW67 MX_SW_solder, SW68 MX_SW_solder, SW69 MX_SW_solder, SW7 MX_SW_solder, SW70 MX_SW_solder, SW71 MX_SW_solder, SW72 MX_SW_solder, SW73 MX_SW_solder, SW74 MX_SW_solder, SW75 MX_SW_solder, SW76 MX_SW_solder, SW77 MX_SW_solder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

Commit message: idk
Parts:
- removed D92: LED_Small, marbastlib-mx:LED_MX_3mm
- removed R4: 220, Resistor_SMD:R_0402_1005Metric
- removed U4: 74AHCT1G125, Package_TO_SOT_SMD:SOT-23-5
- added C14: 100nF, Capacitor_SMD:C_0402_1005Metric, B.Cu at (336.7, 84.5)
- added D94: PRTR5V0U2X, Package_TO_SOT_SMD:SOT-143, B.Cu at (300.0, 27.2)
- added R7: 10k, Resistor_SMD:R_0402_1005Metric, B.Cu at (336.7, 83.4)
- added S7: MX_stab, marbastlib-mx:STAB_MX_10u, B.Cu at (155.2, 126.9)
- SW52: footprint marbastlib-mx:SW_MX_1.75u -> marbastlib-mx:SW_MX_1.75u_STP_1.25
- SW53: footprint marbastlib-mx:SW_MX_1.75u_STP_1.25 -> marbastlib-mx:SW_MX_1.75u
- U3: value SRV05-4 -> TXS0101DBV; footprint marbastlib-various:SOT-23-6-routable -> Package_TO_SOT_SMD:SOT-23-6
- moved U3 67.1 mm to (333.6, 83.4), turned to 0 degrees
- moved C13 26.4 mm to (330.8, 84.8), turned to -90 degrees
- moved C12 5.22 mm to (341.8, 91.3), turned to 0 degrees
- moved R6 5.17 mm to (341.8, 92.4), turned to 180 degrees
- moved R5 5.17 mm to (341.8, 90.1), turned to 0 degrees
- moved SW54 4.74 mm to (55.3, 88.8)
- moved SW55 4.73 mm to (74.3, 88.8)
- moved SW56 4.72 mm to (93.3, 88.8)
- moved SW57 4.71 mm to (112.3, 88.8)
- moved SW58 4.70 mm to (131.3, 88.8)
- moved SW47 4.70 mm to (259.7, 69.8)
- moved SW60 4.70 mm to (169.4, 88.8)
- moved SW59 4.70 mm to (150.4, 88.8)
- moved SW61 4.70 mm to (188.4, 88.8)
- moved C3 4.70 mm to (314.5, 83.2)
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Connections:
- C13 pad 1: +5V -> GND
- C13 pad 2: GND -> +3V3
- J1 pad 2: RGB_DB -> RGBLED
- J3 pad 2: RGB_DB -> RGBLED
- J4 pad 2: RGB_DB -> RGBLED
- U2 pad 26: NUMLOCKLED -> ROW2
- U2 pad 27: ROW2 -> ROW5
- U2 pad 28: ROW5 -> RGB_3V3
- U2 pad 45: RGBLED -> ROW4
- U2 pad 46: ROW4 -> unconnected-(U2-PB9-Pad46)
- U3 pad 1: D+ -> +3V3
- U3 pad 3: unconnected-(U3-IO2-Pad3) -> RGB_3V3
- U3 pad 4: unconnected-(U3-IO3-Pad4) -> RGBLED
- U3 pad 5: VBUS -> Net-(U3-OE)
- U3 pad 6: D- -> +5V
Routing:
- net NUMLOCKLED: track 343.5 -> 0.00 mm
- net COL16: track 149.6 -> 125.6 mm, vias 0 -> 1
- net RGB_3V3: track 0.00 -> 19.3 mm, vias 0 -> 2
- net +3V3: track 72.6 -> 88.9 mm
- net GND: track 69.9 -> 54.2 mm, vias 17 -> 16
- net RGB_DB: track 13.8 -> 0.00 mm
- net COL0: track 416.8 -> 421.6 mm
- net ROW2: track 347.3 -> 351.3 mm
- net COL9: track 238.0 -> 241.4 mm
- net Net-(D92-A): track 3.36 -> 0.00 mm
- net CAPS_LED: track 413.9 -> 417.2 mm
- net COL15: track 202.6 -> 199.4 mm
- net VBUS: track 18.6 -> 21.3 mm
- net COL12: track 187.3 -> 184.6 mm
- net COL13: track 175.5 -> 172.9 mm
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Other:
- board text removed: "C1"
- board text removed: "C5"
- board text removed: "RESET"

Commit message: sunday at the waterpark
Parts:
- removed C13, C14: 100nF, Capacitor_SMD:C_0402_1005Metric
- removed R7: 10k, Resistor_SMD:R_0402_1005Metric
- U3: value TXS0101DBV -> SN74LVC1T45DBV; footprint Package_TO_SOT_SMD:SOT-23-6 -> marbastlib-various:SOT-23-6-routable
- moved U3 0.82 mm to (334.2, 84.1)
Connections:
- U3 pad 5: Net-(U3-OE) -> +3V3
Routing:
- net +3V3: track 88.9 -> 82.0 mm
- net GND: track 54.2 -> 50.7 mm, vias 16 -> 14
- net Net-(U3-OE): track 1.40 -> 0.00 mm
- net RGB_3V3: track 19.3 -> 20.1 mm
- net RGBLED: track 46.1 -> 46.7 mm
