File: pcb/1_2og_repro.kicad_sch (KiCad schematic)
At the start: 29 parts, among them J1 Pico EzMate, J2 548190519, J3 RAW, J4 S3B, Q1 2N7002, SW95 SW_Push, U1 XC6206PxxxMR, U2 STM32F072C8Tx, U3 SRV05-4, U4 74AHCT1G125

Commit message: update gerbers, change mounting hole dimensions
Parts:
- H1, H2: footprint MountingHole:MountingHole_3.2mm_M3_Pad -> MountingHole:MountingHole_3mm_Pad
Changed lines of the file:
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@@
       (effects (font (size 1.27 1.27)) (justify left) hide)
     )
-    (property "Footprint" "MountingHole:MountingHole_3.2mm_M3_Pad" (at 165.227 19.304 0)
+    (property "Footprint" "MountingHole:MountingHole_3mm_Pad" (at 165.227 19.304 0)
       (effects (font (size 1.27 1.27)) hide)
     )
@@
       (effects (font (size 1.27 1.27)) (justify right) hide)
     )
-    (property "Footprint" "MountingHole:MountingHole_3.2mm_M3_Pad" (at 170.307 19.304 0)
+    (property "Footprint" "MountingHole:MountingHole_3mm_Pad" (at 170.307 19.304 0)
       (effects (font (size 1.27 1.27)) hide)
     )

Commit message: ok juggle a few pins around
Connections:
- net RGBLED: now also U2.45 (PB8); no longer U2.2 (PC13)
- net ROW2: now also U2.27 (PB14); no longer U2.37 (PA14)
- net ROW4: now also U2.46 (PB9); no longer U2.3 (PC14)
- net ROW5: now also U2.28 (PB15); no longer U2.4 (PC15)
- no-connect marks 8 -> 11
Other:
- moved on the sheet: U2

Commit message: tune differential pair, reroute to remove redundant vias
Connections:
- net D+: now also U3.1 (IO1); no longer U3.3 (IO2)
- net D-: now also U3.6 (IO4); no longer U3.4 (IO3)
Changed lines of the file:
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@@
   (no_connect (at 60.96 72.39))
   (no_connect (at 27.94 44.45))
-  (no_connect (at 78.867 70.104))
+  (no_connect (at 78.867 75.184))
   (no_connect (at 60.96 85.09))
   (no_connect (at 27.94 41.91))
@@
   (no_connect (at 26.543 107.823))
   (no_connect (at 60.96 82.55))
-  (no_connect (at 104.267 75.184))
+  (no_connect (at 104.267 70.104))
   (no_connect (at 60.96 74.93))
   (wire (pts (xy 75.057 18.669) (xy 85.217 18.669))
@@
     )
   )
-  (global_label "D-" (shape input) (at 104.267 70.104 0) (fields_autoplaced)
+  (global_label "D-" (shape input) (at 104.267 75.184 0) (fields_autoplaced)
     (effects (font (size 1.27 1.27)) (justify left))
-    (property "Intersheetrefs" "${INTERSHEET_REFS}" (at 109.5225 70.0246 0)
+    (property "Intersheetrefs" "${INTERSHEET_REFS}" (at 110.0152 75.184 0)
       (effects (font (size 1.27 1.27)) (justify left) hide)
     )
   )
-  (global_label "D+" (shape input) (at 78.867 75.184 180) (fields_autoplaced)
+  (global_label "D+" (shape input) (at 78.867 70.104 180) (fields_autoplaced)
     (effects (font (size 1.27 1.27)) (justify right))
-    (property "Intersheetrefs" "${INTERSHEET_REFS}" (at 73.6115 75.1046 0)
+    (property "Intersheetrefs" "${INTERSHEET_REFS}" (at 73.1188 70.104 0)
       (effects (font (size 1.27 1.27)) (justify right) hide)
     )

Commit message: idk
Parts:
- removed U3: SRV05-4, marbastlib-various:SOT-23-6-routable, symbol Power_Protection:SRV05-4
- removed U4: 74AHCT1G125, Package_TO_SOT_SMD:SOT-23-5, symbol 74xGxx:74AHCT1G125
- added C14: 100nF, Capacitor_SMD:C_0402_1005Metric, symbol Device:C_Small
- added D94: PRTR5V0U2X, Package_TO_SOT_SMD:SOT-143, symbol Power_Protection:PRTR5V0U2X
- added R7: 10k, Resistor_SMD:R_0402_1005Metric, symbol Device:R_Small
- added U3: TXS0101DBV, Package_TO_SOT_SMD:SOT-23-6, symbol Logic_LevelTranslator:TXS0101DBV
- C13: LCSC C1525 -> (none)
Connections:
- net NUMLOCKLED is gone; now on net ROW2: U2.26 (PB13)
- net RGB_DB is gone; now on net RGBLED: J1.2 (Pin_2), J3.2 (Pin_2), J4.2 (Pin_2)
- net +3V3: now also C13.2, R7.1, U3.1 (V_{CCA})
- net +5V: now also C14.2, U3.6 (V_{CCB}); no longer C13.1
- net D+: now also D94.2 (I/O1)
- net D-: now also D94.3 (I/O2)
- net GND: now also C13.1, C14.1, D94.1 (GND), U3.2 (GND); no longer C13.2
- net RGBLED: now also U3.4 (B); no longer U2.45 (PB8)
- net ROW2: no longer U2.27 (PB14)
- net ROW4: now also U2.45 (PB8); no longer U2.46 (PB9)
- net ROW5: now also U2.27 (PB14); no longer U2.28 (PB15)
- net VBUS: now also D94.4 (VCC)
- new net: R7.2, U3.5 (OE)
- new net RGB_3V3: U2.28 (PB15), U3.3 (A)
- no-connect marks 11 -> 9
Other:
- note added: "Level Shifting"
- note removed: "RGB DB 3.3v->5v"

Commit message: sunday at the waterpark
Parts:
- removed C13, C14: 100nF, Capacitor_SMD:C_0402_1005Metric, symbol Device:C_Small
- removed R7: 10k, Resistor_SMD:R_0402_1005Metric, symbol Device:R_Small
- removed U3: TXS0101DBV, Package_TO_SOT_SMD:SOT-23-6, symbol Logic_LevelTranslator:TXS0101DBV
- added U3: SN74LVC1T45DBV, Package_TO_SOT_SMD:SOT-23-6, symbol Logic_LevelTranslator:SN74LVC1T45DBV
Connections:
- net +3V3: now also U3.1 (VCCA), U3.5 (DIR)
- net +5V: now also U3.6 (VCCB)
- net GND: now also U3.2 (GND)
- net RGBLED: now also U3.4 (B)
- net RGB_3V3: now also U3.3 (A)
