File: pcb/Matrix.kicad_sch (KiCad schematic)
At the start: 196 parts, among them SW1 MX_SW_solder, SW10 MX_SW_solder, SW11 MX_SW_solder, SW12 MX_SW_solder, SW13 MX_SW_solder, SW14 MX_SW_solder, SW15 MX_SW_solder, SW16 MX_SW_solder, SW17 MX_SW_solder, SW18 MX_SW_solder, SW19 MX_SW_solder, SW2 MX_SW_solder, SW20 MX_SW_solder, SW21 MX_SW_solder, SW22 MX_SW_solder, SW23 MX_SW_solder, SW24 MX_SW_solder, SW25 MX_SW_solder, SW26 MX_SW_solder, SW27 MX_SW_solder, SW28 MX_SW_solder, SW29 MX_SW_solder, SW3 MX_SW_solder, SW30 MX_SW_solder, SW31 MX_SW_solder, SW32 MX_SW_solder, SW33 MX_SW_solder, SW34 MX_SW_solder, SW35 MX_SW_solder, SW36 MX_SW_solder, SW37 MX_SW_solder, SW38 MX_SW_solder, SW39 MX_SW_solder, SW4 MX_SW_solder, SW40 MX_SW_solder, SW41 MX_SW_solder, SW42 MX_SW_solder, SW43 MX_SW_solder, SW44 MX_SW_solder, SW45 MX_SW_solder, SW46 MX_SW_solder, SW47 MX_SW_solder, SW48 MX_SW_solder, SW49 MX_SW_solder, SW5 MX_SW_solder, SW50 MX_SW_solder, SW51 MX_SW_solder, SW52 MX_SW_solder, SW53 MX_SW_solder, SW54 MX_SW_solder, SW55 MX_SW_solder, SW56 MX_SW_solder, SW57 MX_SW_solder, SW58 MX_SW_solder, SW59 MX_SW_solder, SW6 MX_SW_solder, SW60 MX_SW_solder, SW61 MX_SW_solder, SW62 MX_SW_solder, SW63 MX_SW_solder, SW64 MX_SW_solder, SW65 MX_SW_solder, SW66 MX_SW_solder, SW67 MX_SW_solder, SW68 MX_SW_solder, SW69 MX_SW_solder, SW7 MX_SW_solder, SW70 MX_SW_solder, SW71 MX_SW_solder, SW72 MX_SW_solder, SW73 MX_SW_solder, SW74 MX_SW_solder, SW75 MX_SW_solder, SW76 MX_SW_solder, SW77 MX_SW_solder, SW78 MX_SW_solder, SW79 MX_SW_solder, SW8 MX_SW_solder, SW80 MX_SW_solder, SW81 MX_SW_solder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

Commit message: idk
Parts:
- removed D92: LED_Small, marbastlib-mx:LED_MX_3mm, symbol Device:LED_Small
- removed R4: 220, Resistor_SMD:R_0402_1005Metric, symbol Device:R_Small
- added S7: MX_stab, marbastlib-mx:STAB_MX_10u, symbol marbastlib-mx:MX_stab
- SW52: renamed from SW53; footprint marbastlib-mx:SW_MX_1.75u -> marbastlib-mx:SW_MX_1.75u_STP_1.25
- SW53: renamed from SW52; footprint marbastlib-mx:SW_MX_1.75u_STP_1.25 -> marbastlib-mx:SW_MX_1.75u
- renumbered D93 to D83, D83 to D84, D84 to D85, D85 to D86, D86 to D87, D87 to D88, D88 to D93, SW92 to SW85, SW85 to SW86, SW93 to SW87, SW94 to SW88, SW86 to SW89, SW87 to SW90, SW88 to SW91, SW89 to SW92, SW90 to SW93, SW91 to SW94
